File: src/KiCad/LittleJimmy/LittleJimmy.kicad_sch (KiCad schematic)
At the start: 9 parts, among them J1 Conn_01x03, J2 Conn_01x04, Q1 BT169B

Commit message: Update to Version 2
Parts:
- Q1: footprint Package_TO_SOT_THT:TO-92_Inline -> Package_TO_SOT_THT:TO-92L_Inline_Wide
Connections:
- net +5V: now also J2.4 (Pin_4); no longer J2.1 (Pin_1)
- net VCC: now also J2.1 (Pin_1); no longer J2.4 (Pin_4)
Changed lines of the file:
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@@
   (title_block
     (title "LittleJimmy")
-    (date "2023-05-13")
-    (rev "0.1")
+    (date "2023-08-03")
+    (rev "2")
     (company "Sebastian Mate")
   )
@@
       (effects (font (size 1.27 1.27)) hide)
     )
-    (property "Value" "VCC" (id 1) (at 22.86 17.78 0))
+    (property "Value" "VCC" (id 1) (at 24.13 17.78 0))
     (property "Footprint" "" (id 2) (at 22.86 22.86 0)
       (effects (font (size 1.27 1.27)) hide)
@@
     (pin "2")
   )
-  (symbol (lib_id "power:VCC") (at 19.05 46.99 0) (unit 1)
-    (in_bom yes) (on_board yes) (fields_autoplaced)
-    (property "Reference" "#PWR02" (id 0) (at 19.05 50.8 0)
-      (effects (font (size 1.27 1.27)) hide)
-    )
-    (property "Value" "VCC" (id 1) (at 19.05 41.91 0))
-    (property "Footprint" "" (id 2) (at 19.05 46.99 0)
-      (effects (font (size 1.27 1.27)) hide)
-    )
-    (property "Datasheet" "" (id 3) (at 19.05 46.99 0)
+  (symbol (lib_id "power:VCC") (at 22.86 46.99 0) (unit 1)
+    (in_bom yes) (on_board yes)
+    (property "Reference" "#PWR02" (id 0) (at 22.86 50.8 0)
+      (effects (font (size 1.27 1.27)) hide)
+    )
+    (property "Value" "VCC" (id 1) (at 24.13 41.91 0))
+    (property "Footprint" "" (id 2) (at 22.86 46.99 0)
+      (effects (font (size 1.27 1.27)) hide)
+    )
+    (property "Datasheet" "" (id 3) (at 22.86 46.99 0)
       (effects (font (size 1.27 1.27)) hide)
     )
@@
       (effects (font (size 1.27 1.27)) (justify left))
     )
-    (property "Footprint" "Package_TO_SOT_THT:TO-92_Inline" (id 2) (at 116.84 38.735 0)
+    (property "Footprint" "Package_TO_SOT_THT:TO-92L_Inline_Wide" (id 2) (at 116.84 38.735 0)
       (effects (font (size 1.27 1.27) italic) (justify left) hide)
     )
@@
     (pin "1")
   )
-  (symbol (lib_id "power:+5V") (at 22.86 46.99 0) (unit 1)
-    (in_bom yes) (on_board yes) (fields_autoplaced)
-    (property "Reference" "#PWR05" (id 0) (at 22.86 50.8 0)
-      (effects (font (size 1.27 1.27)) hide)
-    )
-    (property "Value" "+5V" (id 1) (at 22.86 41.91 0))
-    (property "Footprint" "" (id 2) (at 22.86 46.99 0)
-      (effects (font (size 1.27 1.27)) hide)
-    )
-    (property "Datasheet" "" (id 3) (at 22.86 46.99 0)
+  (symbol (lib_id "power:+5V") (at 19.05 46.99 0) (unit 1)
+    (in_bom yes) (on_board yes) (fields_autoplaced)
+    (property "Reference" "#PWR05" (id 0) (at 19.05 50.8 0)
+      (effects (font (size 1.27 1.27)) hide)
+    )
+    (property "Value" "+5V" (id 1) (at 19.05 41.91 0))
+    (property "Footprint" "" (id 2) (at 19.05 46.99 0)
+      (effects (font (size 1.27 1.27)) hide)
+    )
+    (property "Datasheet" "" (id 3) (at 19.05 46.99 0)
       (effects (font (size 1.27 1.27)) hide)
     )
@@
     )
     (path "/8b1305ce-15af-4e25-bac3-6a32a6576756"
-      (reference "Q1") (unit 1) (value "BT169B") (footprint "Package_TO_SOT_THT:TO-92_Inline")
+      (reference "Q1") (unit 1) (value "BT169B") (footprint "Package_TO_SOT_THT:TO-92L_Inline_Wide")
     )
     (path "/4a62f0d1-abe7-48ee-a9fd-ba32607582fd"
